File: MULTIWII.sch (EAGLE design)
At the start: 30 parts, among them IC1 MEGA8-PU, Q1 16MHz, Q2 BSS138, Q3 BSS138, U1 BMP180

Commit message: first commit
Parts:
- added LED1, LED2: (no value), led:LEDCHIP-LED0603
- added R3, R4, R5, R6: 10K, rcl:R-EU_M0805
Connections:
- net 3.3V: now also R5.2, R6.2
- net 5V: now also R3.2, R4.2
- net GND: now also LED1.C, LED2.C
- net RX: now also LED1.A
- net SCL: now also R6.1
- net SCL0: now also R3.1
- net SDA: now also R5.1
- net SDA0: now also R4.1
- net TX: now also LED2.A
Changed lines of the file:
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@@
 <part name="SJ1" library="Eagle-JeeLabs" deviceset="SOLDERJUMPER" device="NC"/>
 <part name="C8" library="rcl" deviceset="CPOL-EU" device="CT7343"/>
+<part name="R3" library="rcl" deviceset="R-EU_" device="M0805" value="10K"/>
+<part name="R4" library="rcl" deviceset="R-EU_" device="M0805" value="10K"/>
+<part name="R5" library="rcl" deviceset="R-EU_" device="M0805" value="10K"/>
+<part name="R6" library="rcl" deviceset="R-EU_" device="M0805" value="10K"/>
+<part name="LED1" library="led" deviceset="LED" device="CHIP-LED0603"/>
+<part name="LED2" library="led" deviceset="LED" device="CHIP-LED0603"/>
 </parts>
 <sheets>
@@
 <instance part="SJ1" gate="1" x="2.54" y="66.04" rot="R180"/>
 <instance part="C8" gate="G$1" x="119.38" y="-7.62" rot="R90"/>
+<instance part="R3" gate="G$1" x="45.72" y="-20.32" rot="R90"/>
+<instance part="R4" gate="G$1" x="45.72" y="-2.54" rot="R90"/>
+<instance part="R5" gate="G$1" x="25.4" y="-2.54" rot="R90"/>
+<instance part="R6" gate="G$1" x="25.4" y="-20.32" rot="R90"/>
+<instance part="LED1" gate="G$1" x="25.4" y="35.56" rot="R90"/>
+<instance part="LED2" gate="G$1" x="25.4" y="33.02" rot="R90"/>
 </instances>
 <busses>
@@
 <segment>
 <pinref part="Q3" gate="G$1" pin="S"/>
-<wire x1="30.48" y1="-25.4" x2="20.32" y2="-25.4" width="0.1524" layer="91"/>
+<wire x1="30.48" y1="-25.4" x2="25.4" y2="-25.4" width="0.1524" layer="91"/>
 <label x="20.32" y="-25.4" size="1.778" layer="95"/>
+<pinref part="R6" gate="G$1" pin="1"/>
+<wire x1="25.4" y1="-25.4" x2="20.32" y2="-25.4" width="0.1524" layer="91"/>
+<junction x="25.4" y="-25.4"/>
 </segment>
 </net>
@@
 <label x="124.46" y="-7.62" size="1.778" layer="95"/>
 </segment>
+<segment>
+<pinref part="LED1" gate="G$1" pin="C"/>
+<pinref part="LED2" gate="G$1" pin="C"/>
+<wire x1="30.48" y1="35.56" x2="30.48" y2="33.02" width="0.1524" layer="91"/>
+</segment>
 </net>
 <net name="SDA" class="0">
@@
 <segment>
 <pinref part="Q2" gate="G$1" pin="S"/>
-<wire x1="30.48" y1="-7.62" x2="20.32" y2="-7.62" width="0.1524" layer="91"/>
+<wire x1="30.48" y1="-7.62" x2="25.4" y2="-7.62" width="0.1524" layer="91"/>
 <label x="20.32" y="-7.62" size="1.778" layer="95"/>
+<pinref part="R5" gate="G$1" pin="1"/>
+<wire x1="25.4" y1="-7.62" x2="20.32" y2="-7.62" width="0.1524" layer="91"/>
+<junction x="25.4" y="-7.62"/>
 </segment>
 </net>
@@
 <wire x1="180.34" y1="50.8" x2="177.8" y2="50.8" width="0.1524" layer="91"/>
 <pinref part="JP2" gate="A" pin="10"/>
+</segment>
+<segment>
+<pinref part="R4" gate="G$1" pin="2"/>
+<wire x1="45.72" y1="2.54" x2="45.72" y2="5.08" width="0.1524" layer="91"/>
+</segment>
+<segment>
+<wire x1="45.72" y1="-17.78" x2="45.72" y2="-15.24" width="0.1524" layer="91"/>
+<pinref part="R3" gate="G$1" pin="2"/>
+<wire x1="45.72" y1="-15.24" x2="45.72" y2="-10.16" width="0.1524" layer="91"/>
+<junction x="45.72" y="-15.24"/>
 </segment>
 </net>
@@
 <wire x1="33.02" y1="-17.78" x2="33.02" y2="-12.7" width="0.1524" layer="91"/>
 </segment>
+<segment>
+<pinref part="R5" gate="G$1" pin="2"/>
+<wire x1="25.4" y1="2.54" x2="25.4" y2="5.08" width="0.1524" layer="91"/>
+</segment>
+<segment>
+<pinref part="R6" gate="G$1" pin="2"/>
+<wire x1="25.4" y1="-15.24" x2="25.4" y2="-12.7" width="0.1524" layer="91"/>
+</segment>
 </net>
 <net name="N$1" class="0">
@@
 <label x="25.4" y="35.56" size="1.778" layer="95"/>
 <pinref part="SV2" gate="1" pin="5"/>
-<wire x1="17.78" y1="35.56" x2="25.4" y2="35.56" width="0.1524" layer="91"/>
+<wire x1="17.78" y1="35.56" x2="22.86" y2="35.56" width="0.1524" layer="91"/>
 <junction x="17.78" y="35.56"/>
+<pinref part="LED1" gate="G$1" pin="A"/>
+<wire x1="22.86" y1="35.56" x2="25.4" y2="35.56" width="0.1524" layer="91"/>
+<junction x="22.86" y="35.56"/>
 </segment>
 </net>
@@
 <pinref part="SV2" gate="1" pin="4"/>
 <wire x1="17.78" y1="33.02" x2="15.24" y2="33.02" width="0.1524" layer="91"/>
-<wire x1="17.78" y1="33.02" x2="25.4" y2="33.02" width="0.1524" layer="91"/>
+<wire x1="17.78" y1="33.02" x2="22.86" y2="33.02" width="0.1524" layer="91"/>
 <label x="25.4" y="33.02" size="1.778" layer="95"/>
+<pinref part="LED2" gate="G$1" pin="A"/>
+<wire x1="22.86" y1="33.02" x2="25.4" y2="33.02" width="0.1524" layer="91"/>
+<junction x="22.86" y="33.02"/>
 </segment>
 </net>
@@
 <segment>
 <pinref part="Q2" gate="G$1" pin="D"/>
-<wire x1="40.64" y1="-7.62" x2="50.8" y2="-7.62" width="0.1524" layer="91"/>
+<wire x1="40.64" y1="-7.62" x2="45.72" y2="-7.62" width="0.1524" layer="91"/>
 <label x="50.8" y="-7.62" size="1.778" layer="95"/>
+<pinref part="R4" gate="G$1" pin="1"/>
+<wire x1="45.72" y1="-7.62" x2="50.8" y2="-7.62" width="0.1524" layer="91"/>
+<junction x="45.72" y="-7.62"/>
 </segment>
 </net>
@@
 <segment>
 <pinref part="Q3" gate="G$1" pin="D"/>
-<wire x1="40.64" y1="-25.4" x2="50.8" y2="-25.4" width="0.1524" layer="91"/>
+<wire x1="40.64" y1="-25.4" x2="45.72" y2="-25.4" width="0.1524" layer="91"/>
 <label x="48.26" y="-25.4" size="1.778" layer="95"/>
-</segment>
-</net>
+<pinref part="R3" gate="G$1" pin="1"/>
+<wire x1="45.72" y1="-25.4" x2="50.8" y2="-25.4" width="0.1524" layer="91"/>
+<junction x="45.72" y="-25.4"/>
+</segment>
+</net>

Commit message: first commit
Parts:
- C8: value (none) -> 100uF
Connections:
- net SCL: no longer SV3.7, SV3.8
- net SCL0: now also SV3.7, SV3.8
- net SDA: no longer SV3.5, SV3.6
- net SDA0: now also SV3.5, SV3.6
Changed lines of the file:
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@@
 <part name="R2" library="rcl" deviceset="R-EU_" device="M0805" value="1K"/>
 <part name="SJ1" library="Eagle-JeeLabs" deviceset="SOLDERJUMPER" device="NC"/>
-<part name="C8" library="rcl" deviceset="CPOL-EU" device="CT7343"/>
+<part name="C8" library="rcl" deviceset="CPOL-EU" device="CT7343" value="100uF"/>
 <part name="R3" library="rcl" deviceset="R-EU_" device="M0805" value="10K"/>
 <part name="R4" library="rcl" deviceset="R-EU_" device="M0805" value="10K"/>
@@
 <sheet>
 <plain>
+<rectangle x1="30.48" y1="55.88" x2="35.56" y2="58.42" layer="91"/>
 </plain>
 <instances>
@@
 </segment>
 <segment>
-<pinref part="SV3" gate="G$1" pin="7"/>
-<wire x1="63.5" y1="17.78" x2="58.42" y2="17.78" width="0.1524" layer="91"/>
-<wire x1="58.42" y1="17.78" x2="73.66" y2="17.78" width="0.1524" layer="91"/>
-<wire x1="73.66" y1="17.78" x2="86.36" y2="17.78" width="0.1524" layer="91"/>
-<pinref part="SV3" gate="G$1" pin="8"/>
-<junction x="58.42" y="17.78"/>
-<label x="86.36" y="17.78" size="1.778" layer="95"/>
-</segment>
-<segment>
 <pinref part="Q3" gate="G$1" pin="S"/>
 <wire x1="30.48" y1="-25.4" x2="25.4" y2="-25.4" width="0.1524" layer="91"/>
@@
 <pinref part="JP4" gate="A" pin="1"/>
 <wire x1="142.24" y1="7.62" x2="142.24" y2="2.54" width="0.1524" layer="91"/>
+<label x="142.24" y="-2.54" size="1.778" layer="95" rot="R90"/>
 </segment>
 <segment>
@@
 <wire x1="43.18" y1="33.02" x2="38.1" y2="33.02" width="0.1524" layer="91"/>
 <label x="38.1" y="33.02" size="1.778" layer="95"/>
-</segment>
-<segment>
-<wire x1="58.42" y1="15.24" x2="73.66" y2="15.24" width="0.1524" layer="91"/>
-<pinref part="SV3" gate="G$1" pin="5"/>
-<wire x1="73.66" y1="15.24" x2="86.36" y2="15.24" width="0.1524" layer="91"/>
-<junction x="73.66" y="15.24"/>
-<pinref part="SV3" gate="G$1" pin="6"/>
-<label x="86.36" y="15.24" size="1.778" layer="95"/>
 </segment>
 <segment>
@@
 <pinref part="JP4" gate="A" pin="2"/>
 <wire x1="144.78" y1="7.62" x2="144.78" y2="2.54" width="0.1524" layer="91"/>
+<label x="144.78" y="-2.54" size="1.778" layer="95" rot="R90"/>
 </segment>
 <segment>
@@
 <pinref part="R4" gate="G$1" pin="2"/>
 <wire x1="45.72" y1="2.54" x2="45.72" y2="5.08" width="0.1524" layer="91"/>
+<label x="45.72" y="2.54" size="1.778" layer="95"/>
 </segment>
 <segment>
@@
 <wire x1="45.72" y1="-15.24" x2="45.72" y2="-10.16" width="0.1524" layer="91"/>
 <junction x="45.72" y="-15.24"/>
+<label x="45.72" y="-10.16" size="1.778" layer="95"/>
 </segment>
 </net>
@@
 <pinref part="R5" gate="G$1" pin="2"/>
 <wire x1="25.4" y1="2.54" x2="25.4" y2="5.08" width="0.1524" layer="91"/>
+<label x="25.4" y="2.54" size="1.778" layer="95"/>
 </segment>
 <segment>
 <pinref part="R6" gate="G$1" pin="2"/>
 <wire x1="25.4" y1="-15.24" x2="25.4" y2="-12.7" width="0.1524" layer="91"/>
+<label x="25.4" y="-12.7" size="1.778" layer="95"/>
 </segment>
 </net>
@@
 <pinref part="JP4" gate="A" pin="5"/>
 <wire x1="152.4" y1="7.62" x2="152.4" y2="2.54" width="0.1524" layer="91"/>
+<label x="152.4" y="-2.54" size="1.778" layer="95" rot="R90"/>
 </segment>
 </net>
@@
 <pinref part="JP4" gate="A" pin="6"/>
 <wire x1="154.94" y1="7.62" x2="154.94" y2="2.54" width="0.1524" layer="91"/>
+<label x="154.94" y="-2.54" size="1.778" layer="95" rot="R90"/>
 </segment>
 </net>
@@
 <pinref part="JP4" gate="A" pin="8"/>
 <wire x1="160.02" y1="7.62" x2="160.02" y2="2.54" width="0.1524" layer="91"/>
+<label x="160.02" y="-2.54" size="1.778" layer="95" rot="R90"/>
 </segment>
 </net>
@@
 <pinref part="JP4" gate="A" pin="7"/>
 <wire x1="157.48" y1="7.62" x2="157.48" y2="2.54" width="0.1524" layer="91"/>
+<label x="157.48" y="-2.54" size="1.778" layer="95" rot="R90"/>
 </segment>
 </net>
@@
 <pinref part="JP4" gate="A" pin="3"/>
 <wire x1="147.32" y1="7.62" x2="147.32" y2="2.54" width="0.1524" layer="91"/>
+<label x="147.32" y="-2.54" size="1.778" layer="95" rot="R90"/>
 </segment>
 </net>
@@
 <pinref part="JP4" gate="A" pin="4"/>
 <wire x1="149.86" y1="7.62" x2="149.86" y2="2.54" width="0.1524" layer="91"/>
+<label x="149.86" y="-2.54" size="1.778" layer="95" rot="R90"/>
 </segment>
 </net>
@@
 <junction x="45.72" y="-7.62"/>
 </segment>
+<segment>
+<pinref part="SV3" gate="G$1" pin="6"/>
+<wire x1="58.42" y1="15.24" x2="73.66" y2="15.24" width="0.1524" layer="91"/>
+<label x="86.36" y="15.24" size="1.778" layer="95"/>
+<pinref part="SV3" gate="G$1" pin="5"/>
+<wire x1="73.66" y1="15.24" x2="83.82" y2="15.24" width="0.1524" layer="91"/>
+<junction x="73.66" y="15.24"/>
+</segment>
 </net>
 <net name="SCL0" class="0">
@@
 <junction x="45.72" y="-25.4"/>
 </segment>
-</net>
+<segment>
+<pinref part="SV3" gate="G$1" pin="8"/>
+<wire x1="58.42" y1="17.78" x2="73.66" y2="17.78" width="0.1524" layer="91"/>
+<label x="86.36" y="17.78" size="1.778" layer="95"/>
+<pinref part="SV3" gate="G$1" pin="7"/>
+<wire x1="73.66" y1="17.78" x2="83.82" y2="17.78" width="0.1524" layer="91"/>
+<junction x="73.66" y="17.78"/>
+</segment>
+</net>

Commit message: modified:   MULTIWII.brd 	modified:   MULTIWII.sch
Parts:
- removed C4: 10nF, rcl:C-EUC0805
- removed C5: 0.1uF, rcl:C-EUC0805
- removed IC1: MEGA8-PU, avr-7:MEGA8-PU
- removed Q1: 16MHz, crystal:CSM-7X-DU
- removed Q2, Q3: BSS138, m-pad-2.1:BSS138
- removed SJ2: SOLDERJUMPERNC, Eagle-JeeLabs:SOLDERJUMPERNC
- removed SJ3: JUMPER, jumper:SJ2W
- removed U$1: MPU-6050, invensense:MPU-6050
- added F1: (no value), m-pad-2.1:FUSEF
- added IC3: MEGA8-AI, avr-7:MEGA8-AI
- added ISP1: AVRISP-6, adafruit:AVRISP-6
- added PCA9306: (no value), SparkFun-DigitalIC:PCA9306
- added R7, R8: 1K, rcl:R-EU_M0805
- added SJ4: JUMPER, jumper:SJ2W
- added SJ5: SOLDERJUMPERNC, Eagle-JeeLabs:SOLDERJUMPERNC
- added STATUSLED: (no value), adafruit:LEDCHIP-LED0805
- added U2: MPU-6000QFN-24, SparkFun-Sensors:MPU-6000QFN-24
- added Y1: 16MHz, m-pad-2.1:RESONATOR-MURATACSTCR_G
- C3: value 2.2nF -> (none); device rcl:C-EUC0805 -> rcl:CPOL-EUA/3216-18R
- C6: value 22PF -> 0.1uF
- C7: value 22PF -> 2.2nF
- LED1, LED2: device led:LEDCHIP-LED0603 -> adafruit:LEDCHIPLED_0805
- RESET_SW: value SPST_TACT-EVQQ2 -> DTS-6; device adafruit:SPST_TACT-EVQQ2 -> switch-tact:DTS-6
Connections:
- net N$5 renamed C1
- removed net N$10: C5.2, U$1.REGOUT
- removed net N$3: SJ3.2, U$1.AD0
- removed net N$4: C3.2, U$1.CPOUT
- new net AD0: SJ4.2, U2.AD0/SDO
- new net AUXCL: U2.AUXCL
- new net AUXDA: U2.AUXDA
- new net CLKOUT: U2.CLKOUT
- new net INT: U2.INT
- new net N$16: SJ5.1, U2.FSYNC
- new net N$17: SJ1.1, U2.CLKIN
- new net N$18: C6.2, U2.REGOUT
- new net RAW: F1.1, JP2.1, JP2.10, JP2.2, JP2.3, JP2.4, JP2.5, JP2.6, JP2.7, JP2.8, JP2.9, SV2.3
- new net SCK: IC3.PB5(SCK), ISP1.SCK, STATUSLED.A
- net 3.3V: now also PCA9306.VREF1, R8.1, SJ4.1, U2.CS, U2.VDD; no longer IC2.OUT, IC2.OUT@1, Q2.G, Q3.G, SJ3.1, U$1.VDD
- net 5V: now also F1.2, IC3.AVCC, IC3.VCC@1, IC3.VCC@2, ISP1.VCC, R7.1; no longer IC1.AVCC, IC1.VCC@1, JP2.1, JP2.10, JP2.2, JP2.3, JP2.4, JP2.5, JP2.6, JP2.7, JP2.8, JP2.9, SV2.3
- net A0: now also IC3.PC0(ADC0); no longer IC1.PC0(ADC0)
- net A1: now also IC3.PC1(ADC1); no longer IC1.PC1(ADC1)
- net A2: now also IC3.PC2(ADC2); no longer IC1.PC2(ADC2)
- net D10: now also IC3.PB2(SS/OC1B); no longer IC1.PB2(SS/OC1B)
- net D11: now also IC3.PB3(MOSI/OC2), ISP1.MOSI; no longer IC1.PB3(MOSI/OC2)
- net D12: now also IC3.PB4(MISO), ISP1.MISO; no longer IC1.PB4(MISO)
- net D2: now also IC3.PD2(INT0); no longer IC1.PD2(INT0)
- net D3: now also IC3.PD3(INT1); no longer IC1.PD3(INT1)
- net D4: now also IC3.PD4(XCK/T0); no longer IC1.PD4(T0/XCK)
- net D5: now also IC3.PD5(T1); no longer IC1.PD5(T1)
- net D6: now also IC3.PD6(AIN0); no longer IC1.PD6(AIN0)
- net D7: now also IC3.PD7(AIN1); no longer IC1.PD7(AIN1)
- net D8: now also IC3.PB0(ICP); no longer IC1.PB0(ICP1)
- net D9: now also IC3.PB1(OC1A); no longer IC1.PB1(OC1A)
- net GND: now also C3.-, IC3.AGND, IC3.GND@1, IC3.GND@2, ISP1.GND, PCA9306.GND, RESET_SW.1, SJ4.3, SJ5.2, STATUSLED.C, U2.GND, Y1.2; no longer C3.1, C4.1, C5.1, IC1.AGND, IC1.GND@1, RESET_SW.P, SJ2.2, SJ3.3, U$1.GND
- net N$1: now also C7.2, U2.CPOUT; no longer SJ1.1, U$1.CLKIN
- net N$11: now also IC3.PB7(XTAL2/TOSC2), Y1.3; no longer C7.2, IC1.PB7(XTAL2/TOSC2), Q1.1
- net N$2: now also C3.+, IC2.OUT, IC2.OUT@1, R8.2; no longer SJ2.1, U$1.FSYNC
- net N$6: now also IC3.PB6(XTAL1/TOSC1), Y1.1; no longer C6.2, IC1.PB6(XTAL1/TOSC1), Q1.2
- net N$9: now also PCA9306.EN, PCA9306.VREF2, R7.2; no longer C4.2, U$1.VLOGIC
- net RESET: now also IC3.PC6(/RESET), ISP1.RST, RESET_SW.3; no longer IC1.PC6(/RESET), RESET_SW.S
- net RX: now also IC3.PD0(RXD); no longer IC1.PD0(RXD)
- net SCL: now also PCA9306.SCL1, U2.SCL/SCLK; no longer Q3.S, U$1.SCL
- net SCL0: now also IC3.PC5(ADC5/SCL), PCA9306.SCL2; no longer IC1.PC5(ADC5/SCL), Q3.D
- net SDA: now also PCA9306.SDA1, U2.SDA/SDI; no longer Q2.S, U$1.SDA
- net SDA0: now also IC3.PC4(ADC4/SDA), PCA9306.SDA2; no longer IC1.PC4(ADC4/SDA), Q2.D
- net TX: now also IC3.PD1(TXD); no longer IC1.PD1(TXD)
